File: kicad/BarebonesAVR-PCB/BarebonesAVR-PCB.sch (KiCad schematic (older format))
At the start: 14 parts, among them IC1 ATMEGA328-A, P1 ISP6PIN, P2 CONN_FTDI_AVR, SW1 SW-PUSH-RND-SMALL, Y1 8 MHz

Commit message: R2 replaced by 0 ohm resistor
Parts:
- R2: value 10K -> 0
Other:
- note added: "Corrected mistake"
Changed lines of the file:
@@
 P 5400 5000
 F 0 "R2" V 5480 5000 50  0000 C CNN
-F 1 "10K" V 5400 5000 50  0000 C CNN
+F 1 "0" V 5400 5000 50  0000 C CNN
 F 2 "Resistors_SMD:R_0805_HandSoldering" V 5330 5000 50  0001 C CNN
 F 3 "" H 5400 5000 50  0000 C CNN
@@
 Text Label 2900 7300 1    60   ~ 0
 TXD
+Text Notes 4450 5050 0    60   ~ 0
+Corrected mistake
+Wire Notes Line
+	5500 4850 5500 5150
+Wire Notes Line
+	5500 5150 4400 5150
+Wire Notes Line
+	4400 5150 4400 4850
+Wire Notes Line
+	4400 4850 5500 4850
 $EndSCHEMATC
